Commit message: Refractored to be modular for compatibility with various RL and POMDP pipelines. Added RL debug script.

File: roomba.urdf (robot description, URDF)
Before this commit: robot isaac_roomba, 6 links, 5 joints
Links:
- added link front_marker; visual box size=0.04 0.04 0.04
Joints:
- added joint front_marker_joint: type fixed, parent base_link, child front_marker, origin xyz=0.175 0.02 0 rpy=0 0 0
- joint left_wheel_joint: origin xyz=0 -0.024 0.1175 rpy=0 0 0 -> xyz=0 -0.024 -0.1175 rpy=0 0 0
- joint lidar_joint: origin xyz=0 0.05 0 rpy=0 0 0 -> xyz=0 0.15 0 rpy=0 0 0
- joint right_wheel_joint: origin xyz=0 -0.024 -0.1175 rpy=0 0 0 -> xyz=0 -0.024 0.1175 rpy=0 0 0
